File: battery-board/battery-board.kicad_sch (KiCad schematic)
At the start: 8 parts, among them J1 Conn_01x02_Male, J2 Conn_01x03, J3 Screw_Terminal_01x01, SW1 RESET

Commit message: updated to a different fuse
Parts:
- F1: footprint Fuse:Fuse_1206_3216Metric_Pad1.42x1.75mm_HandSolder -> project:Fuse_2920_7451Metric_Pad2.10x5.45mm_HandSolder
Changed lines of the file:
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@@
 			)
 		)
-		(property "Footprint" "Fuse:Fuse_1206_3216Metric_Pad1.42x1.75mm_HandSolder"
+		(property "Footprint" "project:Fuse_2920_7451Metric_Pad2.10x5.45mm_HandSolder"
 			(at 119.38 87.63 0)
 			(effects
